File: Sch1.sch (EAGLE design)
At the start: 110 parts, among them IC101 IR2101, IC102 IR2101, IC103 IR2101, Q101 IRFZ44N, Q102 IRFZ44N, Q103 IRFZ44N, Q104 IRFZ44N, Q105 IRFZ44N, Q106 IRFZ44N, U101 MCP6022-I/SN

Commit message: Köklü Değişiklikler
Çoğu malzeme, özellikle MOSFET'ler ve dirençler SMD formata çevrildi.
Parts:
- added JP103, JP104, JP105, JP106, JP107, JP108, JP109: (no value), pinhead:PINHD-1X1
- added X101: 5202-05-N-02, con-ebyelectro:5202-05-N-02
- C115: device rcl:C-EU050-024X044 -> rcl:C-EU050-025X075
- D101, D102, D103, D104, D105, D106: value 1N5819-T -> SK26; device diode:1N5819-T -> diode:SCHOTTKY-DIODEDO214AA
- D107, D108, D109, D110, D111, D112: device diode:1N4148DO35-7 -> diode:1N4148SOD123
- IC101, IC102, IC103: value IR2101 -> IR2101SMD; device ir2101:IR2101 -> ir2101:IR2101SMD
- Q101, Q102, Q103, Q104, Q105, Q106: value IRFZ44N -> IRFR024; device irfz44n:IRFZ44N -> irfz44n:IRFR024
- R101, R102, R103, R104, R105, R106: device rcl:R-EU_0309/10 -> rcl:R-EU_R0805
- R107, R108, R109, R110, R111, R112, R113, R114, R115, R116, R117, R118, R119, R120, R121, R122, R123, R124, R125, R126, R127: device resistor:R-EU_0309/12 -> resistor:R-EU_R0805
- R132, R133, R134, R135, R136, R137, R138, R139, R140, R141, R142, R143, R144, R145, R146, R147, R148, R149, R150, R151, R152, R153, R154, R155: device rcl:R-EU_0411/12 -> rcl:R-EU_R0805
- R156, R157, R158, R159, R160, R161, R162, R163, R164, R165, R166, R167, R168, R169, R170, R171: device rcl:R-EU_0309/12 -> rcl:R-EU_R0805
Connections:
- removed net N$24: C107.1, Q103.S, Q104.D, R117.2, R124.1, R134.1, R140.1, R146.1, R152.1, R158.2
- removed net N$38: C109.1, Q105.S, Q106.D, R120.2, R126.1, R136.1, R142.1, R148.1, R154.1, R160.2
- removed net N$8: C105.1, Q101.S, Q102.D, R114.2, R122.1, R132.1, R138.1, R144.1, R150.1, R156.2
- new net MOT_A: C105.1, Q101.S, Q102.D, R114.2, R122.1, R132.1, R138.1, R144.1, R150.1, R156.2, X101-1.1
- new net MOT_B: C107.1, Q103.S, Q104.D, R117.2, R124.1, R134.1, R140.1, R146.1, R152.1, R158.2, X101-2.1
- new net MOT_C: C109.1, Q105.S, Q106.D, R120.2, R126.1, R136.1, R142.1, R148.1, R154.1, R160.2, X101-3.1
- net GND: now also X101-4.1
- net ISEN_A: now also JP108.1
- net ISEN_B: now also JP109.1
- net I_A: now also JP106.1
- net I_B: now also JP107.1
- net N$12: no longer D108.C
- net N$5: no longer D108.A
- net VBUS: now also X101-5.1
- net VSEN_A: now also JP103.1
- net VSEN_B: now also JP104.1
- net VSEN_C: now also JP105.1
Other:
- moved on the sheet: C110, C111, C112, C113, C114, C115, R162, R163, R164, R165, R166, R167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

Commit message: Major updates.
Gerber files added.
Scheme and BOM updated.
Parts:
- removed C110, C111, C112, C113: 100pF, rcl:C-EU025-024X044
- removed C114: 1uF, rcl:CPOL-EUE2.5-5
- removed C115: 100nF, rcl:C-EU050-025X075
- removed JP104, JP105, JP106, JP107, JP108, JP109: (no value), pinhead:PINHD-1X1
- removed R152, R153, R154, R155: 1R, rcl:R-EU_R0805
- removed R156, R157, R158, R159, R160, R161: (no value), rcl:R-EU_R0805
- removed R162, R163: 1k, rcl:R-EU_R0805
- removed R164, R166: 27k, rcl:R-EU_R0805
- removed R165, R167: 3.9k, rcl:R-EU_R0805
- removed R168, R169: 1.8k, rcl:R-EU_R0805
- removed R170, R171: 30k, rcl:R-EU_R0805
- removed X101: 5202-05-N-02, con-ebyelectro:5202-05-N-02
- C101, C102, C103: device rcl:CPOL-EUE2.5-5 -> rcl:CPOL-EUSMCA
- C104, C105, C106, C107: value 22nF -> 100pF; device rcl:C-EU050-025X075 -> rcl:C-EUC0805
- C108: value 22nF -> 1uF; device rcl:C-EU050-025X075 -> rcl:CPOL-EUSMCA
- C109: value 22nF -> 100nF; device rcl:C-EU050-025X075 -> rcl:C-EUC1206
- JP102: value OUT -> (none); device pinhead:PINHD-1X7 -> pinhead:PINHD-1X4
- JP103: device pinhead:PINHD-1X1 -> pinhead:PINHD-1X4
- Q101, Q102, Q103, Q104, Q105, Q106: value IRFR024 -> IXTY64N055T; device irfz44n:IRFR024 -> tr:IXTY64N055T
- R132, R133: value 1R -> 0.01; device rcl:R-EU_R0805 -> rcl:R-EU_R2512
- R134, R135, R136, R137, R138, R139, R150, R151: value 1R -> (none)
- R140, R141: value 1R -> 1k
- R142, R144: value 1R -> 27k
- R143, R145: value 1R -> 3.9k
- R146, R147: value 1R -> 1.8k
- R148, R149: value 1R -> 30k
Connections:
- removed net N$12: R108.2
- removed net N$15: C104.2, R132.2, R138.2, R144.2, R150.2
- removed net N$29: C107.2, R135.2, R141.2, R147.2, R153.2
- removed net N$30: C106.2, R134.2, R140.2, R146.2, R152.2
- removed net N$42: C109.2, R137.2, R143.2, R149.2, R155.2
- removed net N$43: C108.2, R136.2, R142.2, R148.2, R154.2
- new net N$8: D108.C, R108.2
- new net VSEN_BUS: JP103.4, R150.1, R151.2
- net +3V3: now also C108.+, C109.1, R142.2, R144.2; no longer C114.+, C115.1, R164.2, R166.2
- net GND: now also C104.2, C105.2, C108.-, C109.2, JP102.4, R129.2, R130.2, R132.2, R133.2, R135.1, R139.1, R145.1, R146.1, R147.1, R151.1; no longer C110.2, C111.2, C114.-, C115.2, JP102.7, Q106.S, R129.1, R130.1, R149.1, R155.1, R157.1, R159.1, R161.1, R165.1, R167.1, R168.1, R169.1, X101-4.1
- net ISEN_A: now also C107.2, JP102.2, R149.2; no longer C113.2, JP102.5, JP108.1, R171.2
- net ISEN_B: now also C106.2, JP102.3, R148.2; no longer C112.2, JP102.6, JP109.1, R170.2
- net I_A: now also R131.2, R140.1; no longer JP106.1, R130.2, R133.1, R139.1, R145.1, R151.1, R162.1
- net I_B: now also R129.1, R132.1; no longer JP107.1, R129.2, R131.2, R135.1, R147.1, R153.1, R163.1
- net MOT_A: now also R134.2; no longer C105.1, R132.1, R138.1, R144.1, R150.1, R156.2, X101-1.1
- net MOT_B: now also R136.2; no longer C107.1, R134.1, R140.1, R146.1, R152.1, R158.2, X101-2.1
- net MOT_C: now also R138.2; no longer C109.1, R136.1, R142.1, R148.1, R154.1, R160.2, X101-3.1
- net N$10: now also C104.1, R141.2, R142.1, R143.2; no longer C110.1, R163.2, R164.1, R165.2
- net N$11: now also C106.1, R146.2, R148.1; no longer C112.1, R168.2, R170.1
- net N$14: now also Q106.S, R130.1, R133.1; no longer C105.2, R133.2, R139.2, R145.2, R151.2
- net N$28: now also C107.1, R147.2, R149.1; no longer C113.1, R169.2, R171.1
- net N$5: now also D108.A
- net N$9: now also C105.1, R140.2, R144.1, R145.2; no longer C111.1, R162.2, R166.1, R167.2
- net VBUS: now also R150.2; no longer C104.1, C106.1, C108.1, X101-5.1
- net VSEN_A: now also R134.1, R135.2; no longer JP102.2, R156.1, R157.2
- net VSEN_B: now also JP103.2, R136.1, R137.2; no longer JP102.3, JP104.1, R158.1, R159.2
- net VSEN_C: now also JP103.3, R138.1, R139.2; no longer JP102.4, JP105.1, R160.1, R161.2
Other:
- moved on the sheet: C104, C105, C106, C107, C109, R129, R130, R131, R132, R133, R134, R135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

Commit message: Last changes before prototyping.
Parts:
- R113, R114, R116, R117, R119, R120: value 10 -> 10R
- R115, R118, R121: value 22 -> 22R
- R134, R136, R138, R150: value (none) -> 68k
- R135, R137, R139, R151: value (none) -> 3.9k
- R143, R145: value 3.9k -> 2.7k
- R146, R147: value 1.8k -> 1.5k
- R148, R149: value 30k -> 27k
Changed lines of the file:
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@@
 <?xml version="1.0" encoding="utf-8"?>
 <!DOCTYPE eagle SYSTEM "eagle.dtd">
-<eagle version="7.6.0">
+<eagle version="7.7.0">
 <drawing>
 <settings>
@@
 <setting verticaltext="up"/>
 </settings>
-<grid distance="0.1" unitdist="inch" unit="inch" style="lines" multiple="1" display="no" altdistance="0.01" altunitdist="inch" altunit="inch"/>
+<grid distance="0.05" unitdist="inch" unit="inch" style="lines" multiple="1" display="no" altdistance="0.01" altunitdist="inch" altunit="inch"/>
 <layers>
 <layer number="1" name="Top" color="4" fill="1" visible="no" active="no"/>
@@
 <parts>
 <part name="U101" library="Microchip_By_element14_Batch_1" deviceset="MCP6022-I/SN" device=""/>
-<part name="R113" library="resistor" deviceset="R-EU_" device="R0805" value="10"/>
-<part name="R115" library="resistor" deviceset="R-EU_" device="R0805" value="22"/>
+<part name="R113" library="resistor" deviceset="R-EU_" device="R0805" value="10R"/>
+<part name="R115" library="resistor" deviceset="R-EU_" device="R0805" value="22R"/>
 <part name="V103" library="supply0" deviceset="+12V" device=""/>
 <part name="GND103" library="supply0" deviceset="GND" device=""/>
@@
 <part name="GND102" library="supply0" deviceset="GND" device=""/>
 <part name="R131" library="rcl" deviceset="R-EU_" device="R2512" value="0.01"/>
-<part name="R149" library="rcl" deviceset="R-EU_" device="R0805" value="30k"/>
+<part name="R149" library="rcl" deviceset="R-EU_" device="R0805" value="27k"/>
 <part name="GND124" library="supply0" deviceset="GND" device=""/>
-<part name="R135" library="rcl" deviceset="R-EU_" device="R0805"/>
-<part name="R134" library="rcl" deviceset="R-EU_" device="R0805"/>
+<part name="R135" library="rcl" deviceset="R-EU_" device="R0805" value="3.9k"/>
+<part name="R134" library="rcl" deviceset="R-EU_" device="R0805" value="68k"/>
 <part name="GND115" library="supply0" deviceset="GND" device=""/>
 <part name="R128" library="rcl" deviceset="R-EU_" device="R2512" value="0.01"/>
@@
 <part name="C109" library="rcl" deviceset="C-EU" device="C1206" value="100nF"/>
 <part name="GND106" library="supply0" deviceset="GND" device=""/>
-<part name="R114" library="resistor" deviceset="R-EU_" device="R0805" value="10"/>
+<part name="R114" library="resistor" deviceset="R-EU_" device="R0805" value="10R"/>
 <part name="C107" library="rcl" deviceset="C-EU" device="C0805" value="100pF"/>
-<part name="R147" library="rcl" deviceset="R-EU_" device="R0805" value="1.8k"/>
+<part name="R147" library="rcl" deviceset="R-EU_" device="R0805" value="1.5k"/>
 <part name="R144" library="rcl" deviceset="R-EU_" device="R0805" value="27k"/>
-<part name="R145" library="rcl" deviceset="R-EU_" device="R0805" value="3.9k"/>
+<part name="R145" library="rcl" deviceset="R-EU_" device="R0805" value="2.7k"/>
 <part name="GND121" library="supply0" deviceset="GND" device=""/>
 <part name="R142" library="rcl" deviceset="R-EU_" device="R0805" value="27k"/>
-<part name="R143" library="rcl" deviceset="R-EU_" device="R0805" value="3.9k"/>
+<part name="R143" library="rcl" deviceset="R-EU_" device="R0805" value="2.7k"/>
 <part name="GND120" library="supply0" deviceset="GND" device=""/>
 <part name="V109" library="supply0" deviceset="+3V3" device=""/>
@@
 <part name="GND119" library="supply0" deviceset="GND" device=""/>
 <part name="GND118" library="supply0" deviceset="GND" device=""/>
-<part name="R146" library="rcl" deviceset="R-EU_" device="R0805" value="1.8k"/>
+<part name="R146" library="rcl" deviceset="R-EU_" device="R0805" value="1.5k"/>
 <part name="GND123" library="supply0" deviceset="GND" device=""/>
-<part name="R148" library="rcl" deviceset="R-EU_" device="R0805" value="30k"/>
+<part name="R148" library="rcl" deviceset="R-EU_" device="R0805" value="27k"/>
 <part name="C106" library="rcl" deviceset="C-EU" device="C0805" value="100pF"/>
 <part name="V111" library="supply0" deviceset="+3V3" device=""/>
@@
 <part name="R123" library="resistor" deviceset="R-EU_" device="R0805" value="4.7k"/>
 <part name="GND109" library="supply0" deviceset="GND" device=""/>
-<part name="R116" library="resistor" deviceset="R-EU_" device="R0805" value="10"/>
-<part name="R118" library="resistor" deviceset="R-EU_" device="R0805" value="22"/>
+<part name="R116" library="resistor" deviceset="R-EU_" device="R0805" value="10R"/>
+<part name="R118" library="resistor" deviceset="R-EU_" device="R0805" value="22R"/>
 <part name="V104" library="supply0" deviceset="+12V" device=""/>
 <part name="GND104" library="supply0" deviceset="GND" device=""/>
@@
 <part name="GND113" library="supply0" deviceset="GND" device=""/>
 <part name="R132" library="rcl" deviceset="R-EU_" device="R2512" value="0.01"/>
-<part name="R137" library="rcl" deviceset="R-EU_" device="R0805"/>
-<part name="R136" library="rcl" deviceset="R-EU_" device="R0805"/>
+<part name="R137" library="rcl" deviceset="R-EU_" device="R0805" value="3.9k"/>
+<part name="R136" library="rcl" deviceset="R-EU_" device="R0805" value="68k"/>
 <part name="GND116" library="supply0" deviceset="GND" device=""/>
 <part name="R129" library="rcl" deviceset="R-EU_" device="R2512" value="0.01"/>
 <part name="GND107" library="supply0" deviceset="GND" device=""/>
-<part name="R117" library="resistor" deviceset="R-EU_" device="R0805" value="10"/>
+<part name="R117" library="resistor" deviceset="R-EU_" device="R0805" value="10R"/>
 <part name="R110" library="resistor" deviceset="R-EU_" device="R0805" value="10R"/>
 <part name="R109" library="resistor" deviceset="R-EU_" device="R0805" value="10R"/>
@@
 <part name="R125" library="resistor" deviceset="R-EU_" device="R0805" value="4.7k"/>
 <part name="GND110" library="supply0" deviceset="GND" device=""/>
-<part name="R119" library="resistor" deviceset="R-EU_" device="R0805" value="10"/>
-<part name="R121" library="resistor" deviceset="R-EU_" device="R0805" value="22"/>
+<part name="R119" library="resistor" deviceset="R-EU_" device="R0805" value="10R"/>
+<part name="R121" library="resistor" deviceset="R-EU_" device="R0805" value="22R"/>
 <part name="V105" library="supply0" deviceset="+12V" device=""/>
 <part name="GND105" library="supply0" deviceset="GND" device=""/>
@@
 <part name="V108" library="supply0" deviceset="VBUS" device=""/>
 <part name="GND114" library="supply0" deviceset="GND" device=""/>
-<part name="R139" library="rcl" deviceset="R-EU_" device="R0805"/>
-<part name="R138" library="rcl" deviceset="R-EU_" device="R0805"/>
+<part name="R139" library="rcl" deviceset="R-EU_" device="R0805" value="3.9k"/>
+<part name="R138" library="rcl" deviceset="R-EU_" device="R0805" value="68k"/>
 <part name="GND117" library="supply0" deviceset="GND" device=""/>
 <part name="GND108" library="supply0" deviceset="GND" device=""/>
-<part name="R120" library="resistor" deviceset="R-EU_" device="R0805" value="10"/>
+<part name="R120" library="resistor" deviceset="R-EU_" device="R0805" value="10R"/>
 <part name="R112" library="resistor" deviceset="R-EU_" device="R0805" value="10R"/>
 <part name="R111" library="resistor" deviceset="R-EU_" device="R0805" value="10R"/>
@@
 <part name="C102" library="rcl" deviceset="CPOL-EU" device="SMCA" value="1uF"/>
 <part name="C101" library="rcl" deviceset="CPOL-EU" device="SMCA" value="1uF"/>
-<part name="R150" library="rcl" deviceset="R-EU_" device="R0805"/>
+<part name="R150" library="rcl" deviceset="R-EU_" device="R0805" value="68k"/>
 <part name="V114" library="supply0" deviceset="VBUS" device=""/>
 <part name="GND127" library="supply0" deviceset="GND" device=""/>
-<part name="R151" library="rcl" deviceset="R-EU_" device="R0805"/>
+<part name="R151" library="rcl" deviceset="R-EU_" device="R0805" value="3.9k"/>
 <part name="JP102" library="pinhead" deviceset="PINHD-1X4" device=""/>
 <part name="JP103" library="pinhead" deviceset="PINHD-1X4" device=""/>
@@
 <instance part="R135" gate="G$1" x="107.95" y="-36.83" rot="R90"/>
 <instance part="R134" gate="G$1" x="107.95" y="-24.13" rot="R90"/>
-<instance part="GND115" gate="1" x="107.95" y="-45.72"/>
+<instance part="GND115" gate="1" x="107.95" y="-46.99"/>
 <instance part="R128" gate="G$1" x="60.96" y="-36.83" rot="R90"/>
 <instance part="V102" gate="G$1" x="-85.09" y="-102.87"/>
@@
 <pinref part="R135" gate="G$1" pin="1"/>
 <pinref part="GND115" gate="1" pin="GND"/>
-<wire x1="107.95" y1="-41.91" x2="107.95" y2="-43.18" width="0.1524" layer="91"/>
-</segment>
-<segment>
+<wire x1="107.95" y1="-41.91" x2="107.95" y2="-44.45" width="0.1524" layer="91"/>
+</segment>
+<segment>
